File: Deprecated/Wheel.kicad_sch (KiCad schematic)
At the start: 44 parts, among them J1 USB_C_Receptacle_USB2.0_16P, J5 Conn_01x06, J6 Conn_01x03, J7 Conn_01x05, SW1 SW_Push, SW2 SW_Push, U1 STM32F407VGTx, U2 AMS1117-3.3

Commit message: Update
Parts:
- removed C11: 4.7µF, Capacitor_SMD:C_0402_1005Metric, symbol Device:C
- added C22: 0.1µF, Capacitor_SMD:C_0805_2012Metric, symbol Device:C
- added R16: 1MΩ, Resistor_SMD:R_0603_1608Metric, symbol Device:R
Connections:
- net +3V3: now also C10.1, C5.1, C6.1, C7.1, C8.1, C9.1, U1.100 (VDD), U1.11 (VDD), U1.19 (VDD), U1.22 (VDDA), U1.28 (VDD), U1.50 (VDD), U1.75 (VDD)
- net GND: now also C10.2, C19.2, C5.2, C6.2, C7.2, C9.2, J1.A1 (GND), J1.A12 (GND), J1.B1 (GND), J1.B12 (GND), C22.2, R16.2
- net at J1.SH (SHIELD): now also C22.1, R16.1
- net at C8.2: no longer U1.50 (VDD)
Other:
- moved on the sheet: C10, C19, C20, C5, C6, C7, C8, C9
