File: Deprecated/untitled - Copy.kicad_sch (KiCad schematic)
At the start: 7 parts, among them J2 Conn_01x06, J3 Conn_01x06, J4 Conn_01x06, U3 MT6835

Commit message: Update
Parts:
- removed J2, J3: Conn_01x06, Connector_PinHeader_2.54mm:PinHeader_1x06_P2.54mm_Vertical, symbol Connector_Generic:Conn_01x06
- added J2, J3: Conn_01x05, Connector_PinHeader_2.54mm:PinHeader_1x05_P2.54mm_Vertical, symbol Connector_Generic:Conn_01x05
Connections:
- net A: now also J2.2 (Pin_2)
- net B: now also J2.3 (Pin_3)
- net CAL: now also J3.5 (Pin_5)
- net GND: now also J2.1 (Pin_1), J3.1 (Pin_1)
- net PWM: now also J2.5 (Pin_5)
- net U: now also J3.2 (Pin_2)
- net V: now also J3.3 (Pin_3)
- net W: now also J3.4 (Pin_4)
- net Z: now also J2.4 (Pin_4)
- net VCC renamed +3V3
