File: Wheel V3/Wheel V3.kicad_sch (KiCad schematic)
At the start: 0 parts

Commit message: Update
Parts:
- added C1, C10, C12, C13, C14, C15, C4, C8, C9: 100nF, symbol Device:C
- added C11, C16, C17, C7: 4.7µF, symbol Device:C
- added C2, C3: 2.2µF, symbol Device:C
- added C5, C6: 15pF, symbol Device:C
- added D1: D_Zener, symbol Device:D_Zener
- added D2: D_Schottky, symbol Device:D_Schottky
- added D3, D4: LED, symbol Device:LED
- added F1: Polyfuse, symbol Device:Polyfuse
- added FB1: 600Ω @ 100MHz, symbol Device:FerriteBead
- added J1: USB_C_Receptacle_USB2.0_16P, symbol Connector:USB_C_Receptacle_USB2.0_16P
- added J10: TEMP, symbol Connector_Generic:Conn_01x02
- added J11: 5V_FanHeader, symbol Connector_Generic:Conn_01x04
- added J12: Conn_01x11, symbol Connector_Generic:Conn_01x11
- added J13: Conn_01x09, symbol Connector_Generic:Conn_01x09
- added J14, J15: Conn_01x07, symbol Connector_Generic:Conn_01x07
- added J16: Conn_01x13, symbol Connector_Generic:Conn_01x13
- added J2: Conn_01x05, symbol Connector_Generic:Conn_01x05
- added J3: Shift Register, symbol Connector_Generic:Conn_01x05
- added J4: MT6835, symbol Connector_Generic:Conn_01x09
- added J5: I2C_Connector, symbol Connector_Generic:Conn_01x07
- added J6: UART_Connector, symbol Connector_Generic:Conn_01x04
- added J7: CAN_Connector, symbol Connector_Generic:Conn_01x04
- added J8: E-Stop, symbol Connector_Generic:Conn_01x02
- added J9: PWM_OUT, symbol Connector_Generic:Conn_01x05
- added R1, R2, R7, R8, R9: 5.1k, symbol Device:R
- added R10, R11, R12, R13: R, symbol Device:R
- added R3, R4: 22, symbol Device:R
- added R5, R6: 10k, symbol Device:R
- added SW1, SW2: SW_Push, symbol Switch:SW_Push
- added U1: STM32F407VGTx, Package_QFP:LQFP-100_14x14mm_P0.5mm, symbol MCU_ST_STM32F4:STM32F407VGTx
- added U2: USBLC6-2SC6, Package_TO_SOT_SMD:SOT-23-6, symbol Power_Protection:USBLC6-2SC6
- added U3: LDL111733R-3.3, Package_TO_SOT_SMD:SOT-223-3_TabPin2, symbol Regulator_Linear:AMS1117-3.3
- added Y1: 8MHz, symbol Device:Crystal_GND24
Connections:
- new net: R5.2, SW1.2, U1.94 (BOOT0)
- new net: J1.B5 (CC2), R1.1
- new net: R3.1, U2.4 (I/O2)
- new net: J10.2 (Pin_2), R12.1, U1.15 (PC0)
- new net: J12.1 (Pin_1), U1.97 (PE0)
- new net: J12.10 (Pin_10), U1.43 (PE12)
- new net: J12.11 (Pin_11), U1.46 (PE15)
- new net: J12.2 (Pin_2), U1.98 (PE1)
- new net: J12.3 (Pin_3), U1.1 (PE2)
- new net: J12.4 (Pin_4), U1.3 (PE4)
- new net: J12.5 (Pin_5), U1.4 (PE5)
- new net: J12.6 (Pin_6), U1.5 (PE6)
- new net: J12.7 (Pin_7), U1.38 (PE7)
- new net: J12.8 (Pin_8), U1.39 (PE8)
- new net: J12.9 (Pin_9), U1.42 (PE11)
- new net: R4.1, U2.6 (I/O1)
- new net: C1.2, J1.SH (SHIELD)
- new net: J13.1 (Pin_1), U1.83 (PD2)
- new net: J13.2 (Pin_2), U1.84 (PD3)
- new net: J13.3 (Pin_3), U1.85 (PD4)
- new net: J13.4 (Pin_4), U1.86 (PD5)
- new net: J13.5 (Pin_5), U1.87 (PD6)
- new net: J13.6 (Pin_6), U1.88 (PD7)
- new net: J13.7 (Pin_7), U1.55 (PD8)
- new net: J13.8 (Pin_8), U1.56 (PD9)
- new net: J13.9 (Pin_9), U1.61 (PD14)
- new net: J1.A5 (CC1), R2.1
- new net: J16.1 (Pin_1), U1.16 (PC1)
- new net: J16.2 (Pin_2), U1.17 (PC2)
- new net: J14.1 (Pin_1), U1.23 (PA0)
- new net: J14.2 (Pin_2), U1.24 (PA1)
- new net: J14.3 (Pin_3), U1.25 (PA2)
- new net: J14.4 (Pin_4), U1.26 (PA3)
- new net: J14.5 (Pin_5), U1.32 (PA7)
- new net: J16.4 (Pin_4), U1.33 (PC4)
- new net: J16.5 (Pin_5), U1.34 (PC5)
- new net: J15.1 (Pin_1), U1.35 (PB0)
- new net: J15.2 (Pin_2), U1.36 (PB1)
- new net: J15.3 (Pin_3), U1.37 (PB2)
- new net: J15.6 (Pin_6), U1.47 (PB10)
- new net: J15.7 (Pin_7), U1.48 (PB11)
- new net: C2.2, U1.49 (VCAP_1)
- new net: J16.6 (Pin_6), U1.65 (PC8)
- new net: J16.7 (Pin_7), U1.66 (PC9)
- new net: J14.6 (Pin_6), U1.67 (PA8)
- new net: J16.11 (Pin_11), U1.7 (PC13)
- new net: C3.2, U1.73 (VCAP_2)
- new net: J14.7 (Pin_7), U1.77 (PA15)
- new net: J16.8 (Pin_8), U1.78 (PC10)
- new net: J16.9 (Pin_9), U1.79 (PC11)
- new net: J16.12 (Pin_12), U1.8 (PC14)
- new net: J16.10 (Pin_10), U1.80 (PC12)
- new net: J15.4 (Pin_4), U1.89 (PB3)
- new net: J16.13 (Pin_13), U1.9 (PC15)
- new net: J15.5 (Pin_5), U1.90 (PB4)
- new net: D1.1 (K), D2.2 (A), F1.2
- new net: D4.2 (A), R11.2
- new net: D3.2 (A), R10.2
- new net +3V3: C10.1, C11.1, C13.1, C14.1, C15.1, C17.1, C7.1, C8.1, C9.1, FB1.1, J16.3 (Pin_3), J2.1 (Pin_1), J3.1 (Pin_1), J4.1 (Pin_1), J5.1 (Pin_1), R10.1, R11.1, R12.2, R13.2, R6.1, R7.1, R8.2, R9.2, SW1.1, U1.100 (VDD), U1.11 (VDD), U1.18 (PC3), U1.19 (VDD), U1.28 (VDD), U1.50 (VDD), U1.6 (VBAT), U1.75 (VDD), U3.2 (VO)
- new net +5V: C16.1, D2.1 (K), J11.2 (Pin_2), J6.1 (Pin_1), J7.1 (Pin_1), U3.3 (VI)
- new net CAN_RX: J7.3 (Pin_3), U1.81 (PD0)
- new net CAN_TX: J7.4 (Pin_4), U1.82 (PD1)
- new net ENC_A: J4.4 (Pin_4), R9.1, U1.63 (PC6)
- new net ENC_B: J4.3 (Pin_3), R8.1, U1.64 (PC7)
- new net ENC_Z: J4.2 (Pin_2), R7.2, U1.62 (PD15)
- new net E_STOP: J8.1 (Pin_1), U1.2 (PE3)
- new net GND: C1.1, C10.2, C11.2, C12.1, C13.2, C14.2, C15.2, C16.2, C17.2, C2.1, C3.1, C4.2, C5.2, C6.2, C7.2, C8.2, C9.2, D1.2 (A), J1.A1 (GND), J1.A12 (GND), J1.B1 (GND), J1.B12 (GND), J10.1 (Pin_1), J11.1 (Pin_1), J2.4 (Pin_4), J3.2 (Pin_2), J4.5 (Pin_5), J5.2 (Pin_2), J6.2 (Pin_2), J7.2 (Pin_2), J8.2 (Pin_2), J9.1 (Pin_1), R1.2, R2.2, R5.1, SW2.1, U1.10 (VSS), U1.20 (VSSA), U1.27 (VSS), U1.74 (VSS), U1.99 (VSS), U2.2 (GND), U3.1 (GND), Y1.2 (G), Y1.4 (G)
- new net I2C_GPIO_1: J5.5 (Pin_5), U1.91 (PB5)
- new net I2C_GPIO_2: J5.6 (Pin_6), U1.92 (PB6)
- new net I2C_GPIO_3: J5.7 (Pin_7), U1.93 (PB7)
- new net I2C_SCL: J5.3 (Pin_3), U1.95 (PB8)
- new net I2C_SDA: J5.4 (Pin_4), U1.96 (PB9)
- new net LED_ERR: D4.1 (K), U1.45 (PE14)
- new net LED_OK: D3.1 (K), U1.44 (PE13)
- new net NRST: C12.2, J2.5 (Pin_5), R6.2, SW2.2, U1.14 (NRST)
- new net OSC+: C5.1, U1.12 (PH0), Y1.1
- new net OSC-: C6.1, U1.13 (PH1), Y1.3
- new net PE10: J11.3 (Pin_3), R13.1, U1.41 (PE10)
- new net PE9: J11.4 (Pin_4), U1.40 (PE9)
- new net PWM1: J9.2 (Pin_2), U1.57 (PD10)
- new net PWM2: J9.3 (Pin_3), U1.58 (PD11)
- new net PWM3: J9.4 (Pin_4), U1.59 (PD12)
- new net PWM4: J9.5 (Pin_5), U1.60 (PD13)
- new net SPI1_CS: J3.5 (Pin_5), U1.29 (PA4)
- new net SPI1_MISO: J3.4 (Pin_4), U1.31 (PA6)
- new net SPI1_SCK: J3.3 (Pin_3), U1.30 (PA5)
- new net SPI2_CS: J4.9 (Pin_9), U1.51 (PB12)
- new net SPI2_MISO: J4.7 (Pin_7), U1.53 (PB14)
- new net SPI2_MOSI: J4.8 (Pin_8), U1.54 (PB15)
- new net SPI2_SCK: J4.6 (Pin_6), U1.52 (PB13)
- new net SWCLK: J2.3 (Pin_3), U1.76 (PA14)
- new net SWDIO: J2.2 (Pin_2), U1.72 (PA13)
- new net UART_RX: J6.4 (Pin_4), U1.69 (PA10)
- new net UART_TX: J6.3 (Pin_3), U1.68 (PA9)
- new net USB_D+: U1.70 (PA11), U2.1 (I/O1)
- new net USB_D+_IN: J1.A6 (D+), J1.B6 (D+), R4.2
- new net USB_D-: U1.71 (PA12), U2.3 (I/O2)
- new net USB_D-_IN: J1.A7 (D-), J1.B7 (D-), R3.2
- new net VBUS: F1.1, J1.A4 (VBUS), J1.A9 (VBUS), J1.B4 (VBUS), J1.B9 (VBUS), U2.5 (VBUS)
- new net VDDA: C4.1, FB1.2, U1.21 (VREF+), U1.22 (VDDA)
- no-connect marks 0 -> 2

Commit message: Update
Parts:
- removed J11: 5V_FanHeader, symbol Connector_Generic:Conn_01x04
- removed J12: Conn_01x11, symbol Connector_Generic:Conn_01x11
- removed J13: Conn_01x09, symbol Connector_Generic:Conn_01x09
- removed J15: Conn_01x07, symbol Connector_Generic:Conn_01x07
- removed J16: Conn_01x13, symbol Connector_Generic:Conn_01x13
- removed R13: R, symbol Device:R
- added J1: Motor_Off, Connector_JST:JST_XH_B2B-XH-A_1x02_P2.50mm_Vertical, symbol Connector_Generic:Conn_01x02
- C1, C10, C7, C8, C9: footprint (none) -> Capacitor_SMD:C_0805_2012Metric
- C11: renamed from C13; footprint (none) -> Capacitor_SMD:C_0805_2012Metric
- C12: renamed from C14; footprint (none) -> Capacitor_SMD:C_0805_2012Metric
- C13: renamed from C15; footprint (none) -> Capacitor_SMD:C_0805_2012Metric
- C14: renamed from C11; footprint (none) -> Capacitor_SMD:C_0805_2012Metric
- C15: renamed from C12; footprint (none) -> Capacitor_SMD:C_0805_2012Metric
- C16: renamed from C2; footprint (none) -> Capacitor_SMD:C_0805_2012Metric
- C17: renamed from C3; footprint (none) -> Capacitor_SMD:C_0805_2012Metric
- C2: renamed from C4; footprint (none) -> Capacitor_SMD:C_0805_2012Metric
- C3: renamed from C5; footprint (none) -> Capacitor_SMD:C_0805_2012Metric
- C4: renamed from C6; footprint (none) -> Capacitor_SMD:C_0805_2012Metric
- C5: renamed from C16; footprint (none) -> Capacitor_SMD:C_0805_2012Metric
- C6: renamed from C17; footprint (none) -> Capacitor_SMD:C_0805_2012Metric
- D1: renamed from D2; footprint (none) -> Diode_SMD:D_SOD-123
- D2: renamed from D1; footprint (none) -> Diode_SMD:D_SOD-123
- D3, D4: footprint (none) -> LED_SMD:LED_0805_2012Metric
- F1: footprint (none) -> Fuse:Fuse_1206_3216Metric
- FB1: footprint (none) -> Inductor_SMD:L_0805_2012Metric
- J10: renamed from J6; footprint (none) -> Connector_JST:JST_XH_B4B-XH-A_1x04_P2.50mm_Vertical
- J12: renamed from J10; footprint (none) -> Connector_JST:JST_XH_B2B-XH-A_1x02_P2.50mm_Vertical
- J13: renamed from J2; footprint (none) -> Connector_JST:JST_XH_B5B-XH-A_1x05_P2.50mm_Vertical
- J15: renamed from J3; footprint (none) -> Connector_JST:JST_XH_B5B-XH-A_1x05_P2.50mm_Vertical
- J16: renamed from J4; footprint (none) -> Connector_JST:JST_XH_B9B-XH-A_1x09_P2.50mm_Vertical
- J2: renamed from J1; footprint (none) -> Connector_USB:USB_C_Receptacle_HRO_TYPE-C-31-M-12
- J3: renamed from J14; footprint (none) -> Connector_JST:JST_XH_B7B-XH-A_1x07_P2.50mm_Vertical
- J4: renamed from J9; footprint (none) -> Connector_JST:JST_XH_B5B-XH-A_1x05_P2.50mm_Vertical
- J6: renamed from J7; footprint (none) -> Connector_JST:JST_XH_B4B-XH-A_1x04_P2.50mm_Vertical
- J8: renamed from J5; footprint (none) -> Connector_JST:JST_XH_B7B-XH-A_1x07_P2.50mm_Vertical
- J9: renamed from J8; footprint (none) -> Connector_JST:JST_XH_B2B-XH-A_1x02_P2.50mm_Vertical
- R1, R2: footprint (none) -> Resistor_SMD:R_0805_2012Metric
- R10: renamed from R7; footprint (none) -> Resistor_SMD:R_0805_2012Metric
- R11: renamed from R8; footprint (none) -> Resistor_SMD:R_0805_2012Metric
- R12: renamed from R9; footprint (none) -> Resistor_SMD:R_0805_2012Metric
- R3: renamed from R5; footprint (none) -> Resistor_SMD:R_0805_2012Metric
- R4: renamed from R3; footprint (none) -> Resistor_SMD:R_0805_2012Metric
- R5: renamed from R4; footprint (none) -> Resistor_SMD:R_0805_2012Metric
- R6: renamed from R10; footprint (none) -> Resistor_SMD:R_0805_2012Metric
- R7: renamed from R11; footprint (none) -> Resistor_SMD:R_0805_2012Metric
- R8: renamed from R12; footprint (none) -> Resistor_SMD:R_0805_2012Metric
- R9: renamed from R6; footprint (none) -> Resistor_SMD:R_0805_2012Metric
- SW1, SW2: footprint (none) -> Button_Switch_SMD:SW_SPST_B3U-1000P
- Y1: footprint (none) -> Crystal:Crystal_SMD_5032-4Pin_5.0x3.2mm
- renumbered U2 to U1, U3 to U2, U1 to U3
Connections:
- net +3V3: no longer R6.1
- net GND: now also J1.2 (Pin_2)
- net PE10: now also J1.1 (Pin_1)
- net PE9: no longer names the net of U3.40 (PE9)
Other:
- added sheet MT6835 (MT6835.kicad_sch)
