File: Wheel V3/Wheel V3.kicad_sch (KiCad schematic)
At the start: 53 parts, among them J1 Motor_Off, J10 UART_Connector, J12 TEMP, J13 Conn_01x05, J15 Shift Register, J16 MT6835, J2 USB_C_Receptacle_USB2.0_16P, J3 Conn_01x07, J4 PWM_OUT, J6 CAN_Connector, J8 I2C_Connector, J9 E-Stop, SW1 SW_Push, SW2 SW_Push, U1 USBLC6-2SC6, U2 LDL111733R-3.3, U3 STM32F407VGTx, Y1 8MHz

Commit message: Update
Parts:
- added R1: 1M, Resistor_SMD:R_0805_2012Metric, symbol Device:R
- added R7, R8: 2.2k, Resistor_SMD:R_0805_2012Metric, symbol Device:R
- C1: value 100nF -> 0.1uF
- renumbered J13 to J10, J15 to J11, J16 to J12, J6 to J5, J8 to J6, J9 to J7, J10 to J8, J12 to J9, R7 to R10, R8 to R11, R9 to R12, R10 to R13, R11 to R14, R12 to R15, R1 to R2, R2 to R3, R3 to R4, R4 to R5, R5 to R6, R6 to R9
Connections:
- net +3V3: now also R9.1, R7.1, R8.1
- net GND: now also C1.2, R1.1; no longer C1.1
- net I2C_SCL: now also R7.2
- net I2C_SDA: now also R8.2
- net at J2.SH (SHIELD): now also C1.1, R1.2; no longer C1.2

Commit message: Update
Parts:
- D3: value LED -> GREEN
- D4: value LED -> RED
- R10, R9: value R -> 1.5k
- R11: value R -> 10k
Changed lines of the file:
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@@
 			)
 		)
-		(property "Value" "R"
+		(property "Value" "10k"
 			(at 101.6 137.1599 0)
 			(hide yes)
@@
 			)
 		)
-		(property "Value" "R"
+		(property "Value" "1.5k"
 			(at 129.54 123.1899 0)
 			(show_name no)
@@
 			)
 		)
-		(property "Value" "LED"
+		(property "Value" "RED"
 			(at 130.81 132.3974 90)
 			(show_name no)
@@
 			)
 		)
-		(property "Value" "R"
+		(property "Value" "1.5k"
 			(at 119.38 123.1899 0)
 			(show_name no)
@@
 			)
 		)
-		(property "Value" "LED"
+		(property "Value" "GREEN"
 			(at 120.65 132.3974 90)
 			(show_name no)

Commit message: Update
Other:
- added sheet Brake (Brake.kicad_sch)
Changed lines of the file:
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@@
+	)
+	(sheet
+		(at 238.76 57.785)
+		(size 31.115 19.685)
+		(exclude_from_sim no)
+		(in_bom yes)
+		(on_board yes)
+		(dnp no)
+		(fields_autoplaced yes)
+		(stroke
+			(width 0.1524)
+			(type solid)
+		)
+		(fill
+			(color 0 0 0 0)
+		)
+		(property "Sheetname" "Brake"
+			(at 238.76 57.0734 0)
+			(show_name no)
+			(do_not_autoplace no)
+			(effects
+				(font
+					(size 1.27 1.27)
+				)
+				(justify left bottom)
+			)
+		)
+		(property "Sheetfile" "Brake.kicad_sch"
+			(at 238.76 78.0546 0)
+			(show_name no)
+			(do_not_autoplace no)
+			(effects
+				(font
+					(size 1.27 1.27)
+				)
+				(justify left top)
+			)
+		)
+		(instances
+			(project "Wheel V3"
+				(path "/9ec62b0c-f2ce-42d9-a60a-bf785e542e97"
+					(page "3")
+				)
+			)
+		)
 	)
 	(sheet

Commit message: Update
Other:
- removed sheet Brake
Changed lines of the file:
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@@
-	)
-	(sheet
-		(at 238.76 57.785)
-		(size 31.115 19.685)
-		(exclude_from_sim no)
-		(in_bom yes)
-		(on_board yes)
-		(dnp no)
-		(fields_autoplaced yes)
-		(stroke
-			(width 0.1524)
-			(type solid)
-		)
-		(fill
-			(color 0 0 0 0)
-		)
-		(property "Sheetname" "Brake"
-			(at 238.76 57.0734 0)
-			(show_name no)
-			(do_not_autoplace no)
-			(effects
-				(font
-					(size 1.27 1.27)
-				)
-				(justify left bottom)
-			)
-		)
-		(property "Sheetfile" "Brake.kicad_sch"
-			(at 238.76 78.0546 0)
-			(show_name no)
-			(do_not_autoplace no)
-			(effects
-				(font
-					(size 1.27 1.27)
-				)
-				(justify left top)
-			)
-		)
-		(instances
-			(project "Wheel V3"
-				(path "/9ec62b0c-f2ce-42d9-a60a-bf785e542e97"
-					(page "3")
-				)
-			)
-		)
 	)
 	(sheet
