File: Wheel V3/MT6835.kicad_sch (KiCad schematic)
At the start: 2 parts, among them IC1 MT6835GT-STD, J17 MT6835

Commit message: Update
Parts:
- renumbered J17 to J13
Changed lines of the file:
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@@
 		(in_pos_files yes)
 		(dnp no)
-		(property "Reference" "J17"
+		(property "Reference" "J13"
 			(at 189.23 58.4199 0)
 			(show_name no)
@@
 			(project "Wheel V3"
 				(path "/9ec62b0c-f2ce-42d9-a60a-bf785e542e97/c571442b-5270-47cf-acbf-8c0f5836bd1c"
-					(reference "J17")
+					(reference "J13")
 					(unit 1)
 				)
@@
 		(dnp no)
 		(fields_autoplaced yes)
-		(property "Reference" "#PWR053"
+		(property "Reference" "#PWR055"
 			(at 167.64 92.71 0)
 			(hide yes)
@@
 			(project "Wheel V3"
 				(path "/9ec62b0c-f2ce-42d9-a60a-bf785e542e97/c571442b-5270-47cf-acbf-8c0f5836bd1c"
-					(reference "#PWR053")
+					(reference "#PWR055")
 					(unit 1)
 				)
@@
 		(dnp no)
 		(fields_autoplaced yes)
-		(property "Reference" "#PWR052"
+		(property "Reference" "#PWR054"
 			(at 175.26 59.69 0)
 			(hide yes)
@@
 			(project "Wheel V3"
 				(path "/9ec62b0c-f2ce-42d9-a60a-bf785e542e97/c571442b-5270-47cf-acbf-8c0f5836bd1c"
-					(reference "#PWR052")
+					(reference "#PWR054")
 					(unit 1)
 				)
