File: Wheel V3/Wheel V3.kicad_pcb (KiCad board)
At the start: 2 copper layers, 148.3 x 76.2 mm, 55 parts, among them IC1 MT6835GT-STD, J1 Motor_Off, J10 UART_Connector, J12 TEMP, J13 Conn_01x05, J15 Shift Register, J16 MT6835, J17 MT6835, J2 USB_C_Receptacle_USB2.0_16P, J3 Conn_01x07, J4 PWM_OUT, J6 CAN_Connector, J8 I2C_Connector, J9 E-Stop, SW1 SW_Push, SW2 SW_Push, U1 USBLC6-2SC6, U2 LDL111733R-3.3, U3 STM32F407VGTx, Y1 8MHz

Commit message: Update
Parts:
- added R1: 1M, Resistor_SMD:R_0805_2012Metric, F.Cu at (218.9, 22.1)
- added R7: 2.2k, Resistor_SMD:R_0805_2012Metric, F.Cu at (157.2, 32.8)
- added R8: 2.2k, Resistor_SMD:R_0805_2012Metric, F.Cu at (162.1, 30.5)
- C1: value 100nF -> 0.1uF
- moved C1 1.41 mm to (218.9, 24.1), turned to 180 degrees
- renumbered J13 to J10, J15 to J11, J16 to J12, J17 to J13, J6 to J5, J8 to J6, J9 to J7, J10 to J8, J12 to J9, R7 to R10, R8 to R11, R9 to R12, R10 to R13, R11 to R14, R12 to R15, R1 to R2, R2 to R3, R3 to R4, R4 to R5, R5 to R6, R6 to R9
Connections:
- C1 pad 1: GND -> Net-(J2-SHIELD)
- C1 pad 2: Net-(J2-SHIELD) -> GND
- R9 pad 1: unconnected-(R6-Pad1) -> +3V3
Routing:
- net +3V3: track 202.7 -> 209.9 mm
- net Net-(J2-SHIELD): track 21.3 -> 25.2 mm
- net GND: track 50.3 -> 47.3 mm
- net I2C_SCL: track 17.9 -> 20.3 mm, vias 1 -> 3
- net I2C_SDA: track 15.9 -> 16.4 mm

Commit message: Update
Parts:
- D3: value LED -> GREEN
- D4: value LED -> RED
- R10, R9: value R -> 1.5k
- R11: value R -> 10k
Changed lines of the file:
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@@
 			(drillshape 0)
 			(scaleselection 1)
-			(outputdirectory "../Production/")
+			(outputdirectory "../Gerbers/")
 		)
 	)
@@
 			)
 		)
-		(property "Value" "LED"
+		(property "Value" "RED"
 			(at 0 1.65 0)
 			(layer "F.Fab")
@@
 			)
 		)
-		(property "Value" "R"
+		(property "Value" "1.5k"
 			(at 0 1.65 0)
 			(layer "F.Fab")
@@
 			)
 		)
-		(property "Value" "LED"
+		(property "Value" "GREEN"
 			(at 0 1.65 0)
 			(layer "F.Fab")
@@
 			)
 		)
-		(property "Value" "R"
+		(property "Value" "10k"
 			(at 0 1.65 0)
 			(layer "F.Fab")
@@
 			)
 		)
-		(property "Value" "R"
+		(property "Value" "1.5k"
 			(at 0 1.65 0)
 			(layer "F.Fab")
