File: Wheel V3/Wheel V3.kicad_pcb (KiCad board)
At the start: 2 copper layers, 148.3 x 76.2 mm, 63 parts, among them IC1 MT6835GT-STD, J1 Motor_Off, J10 Conn_01x05, J11 Shift Register, J12 MT6835, J13 MT6835, J2 USB_C_Receptacle_USB2.0_16P, J3 Conn_01x07, J4 PWM_OUT, J5 CAN_Connector, J6 I2C_Connector, J7 E-Stop, J8 UART_Connector, J9 TEMP, SW1 SW_Push, SW2 SW_Push, U1 USBLC6-2SC6, U2 LDL111733R-3.3, U3 STM32F407VGTx, Y1 8MHz

Commit message: Update
Parts:
- removed MB5 (x5): 5.5mm, PCM_marbastlib-various:mousebites_5p5mm_easysnap
- added C18: 10uF, Capacitor_SMD:C_0805_2012Metric, F.Cu at (93.7, 27.4)
- added C19: 10uF, Capacitor_SMD:C_0805_2012Metric, F.Cu at (136.1, 25.1)
- added C20: 100nF, Capacitor_SMD:C_0805_2012Metric, F.Cu at (136.1, 27.2)
- added C21: 100nF, Capacitor_SMD:C_0805_2012Metric, F.Cu at (136.1, 29.2)
- added J14: PWR, Connector_AMASS:AMASS_XT60-M_1x02_P7.20mm_Vertical, F.Cu at (93.6, 33.8)
- added J15: Resistor, Connector_AMASS:AMASS_XT60-M_1x02_P7.20mm_Vertical, F.Cu at (102.4, 45.7)
- added Q1: STP110N8F6, Package_TO_SOT_THT:TO-220-3_Vertical, F.Cu at (112.3, 45.1)
- added R16: 100k, Resistor_SMD:R_0805_2012Metric, F.Cu at (104.9, 27.2)
- added R17: 10k, Resistor_SMD:R_0805_2012Metric, F.Cu at (101.4, 25.1)
- added R18: 10k, Resistor_SMD:R_0805_2012Metric, F.Cu at (110.5, 22.9)
- added R19: 10k, Resistor_SMD:R_0805_2012Metric, F.Cu at (104.9, 25.1)
- added U4: L7812, Converter_DCDC:Converter_DCDC_RECOM_R-78E-0.5_THT, F.Cu at (125.6, 28.9)
- added U5: LM393, Package_SO:SOIC-8_3.9x4.9mm_P1.27mm, F.Cu at (110.5, 26.7)
- added U6: TL431D, Package_SO:SOIC-8_3.9x4.9mm_P1.27mm, F.Cu at (116.8, 32.3)
- added U7: TC4427xOA, Package_SO:SOIC-8_3.9x4.9mm_P1.27mm, F.Cu at (109.4, 37.5)
Routing:
- net +12V: track 0.00 -> 62.4 mm
- net +24V: track 0.00 -> 58.1 mm, vias 0 -> 4
- net Net-(U7-IN_A): track 0.00 -> 28.9 mm
- net Net-(J15-Pin_1): track 0.00 -> 13.2 mm
- net Net-(U5A--): track 0.00 -> 10.7 mm
- net Net-(Q1-G): track 0.00 -> 10.3 mm
- net Net-(U5A-+): track 0.00 -> 8.37 mm

Commit message: Update
Parts:
- removed C18, C19: 10uF, Capacitor_SMD:C_0805_2012Metric
- removed C20, C21: 100nF, Capacitor_SMD:C_0805_2012Metric
- removed J14: PWR, Connector_AMASS:AMASS_XT60-M_1x02_P7.20mm_Vertical
- removed J15: Resistor, Connector_AMASS:AMASS_XT60-M_1x02_P7.20mm_Vertical
- removed Q1: STP110N8F6, Package_TO_SOT_THT:TO-220-3_Vertical
- removed R16: 100k, Resistor_SMD:R_0805_2012Metric
- removed R17, R18, R19: 10k, Resistor_SMD:R_0805_2012Metric
- removed U4: L7812, Converter_DCDC:Converter_DCDC_RECOM_R-78E-0.5_THT
- removed U5: LM393, Package_SO:SOIC-8_3.9x4.9mm_P1.27mm
- removed U6: TL431D, Package_SO:SOIC-8_3.9x4.9mm_P1.27mm
- removed U7: TC4427xOA, Package_SO:SOIC-8_3.9x4.9mm_P1.27mm
Routing:
- net +12V: track 62.4 -> 0.00 mm
- net +24V: track 58.1 -> 0.00 mm, vias 4 -> 0
- net Net-(U7-IN_A): track 28.9 -> 0.00 mm
- net Net-(J15-Pin_1): track 13.2 -> 0.00 mm
- net Net-(U5A--): track 10.7 -> 0.00 mm
- net Net-(Q1-G): track 10.3 -> 0.00 mm
- net Net-(U5A-+): track 8.37 -> 0.00 mm

Commit message: Final Update
Parts:
- added REF**: MouseBite-Slot_2.0x4.5mm_outset_D0.5mm_P0.85mm_7h, Panelization:MouseBite-Slot_2.0x4.5mm_outset_D0.5mm_P0.85mm_7h, F.Cu at (199.4, 78.1)
- added REF**: MouseBite-Slot_2.0x4.5mm_outset_D0.5mm_P0.85mm_7h, Panelization:MouseBite-Slot_2.0x4.5mm_outset_D0.5mm_P0.85mm_7h, F.Cu at (217.4, 61.2)
- added REF**: MouseBite-Slot_2.0x4.5mm_outset_D0.5mm_P0.85mm_7h, Panelization:MouseBite-Slot_2.0x4.5mm_outset_D0.5mm_P0.85mm_7h, F.Cu at (199.4, 71.2)
- added REF**: MouseBite-Slot_2.0x4.5mm_outset_D0.5mm_P0.85mm_7h, Panelization:MouseBite-Slot_2.0x4.5mm_outset_D0.5mm_P0.85mm_7h, F.Cu at (224.3, 61.2)
- moved IC1 117.4 mm to (215.9, 65.7), turned to 180 degrees
- moved J13 93.2 mm to (204.7, 77.1), turned to 0 degrees
- moved J7 9.40 mm to (140.2, 42.0)
- moved J9 9.14 mm to (140.0, 50.8)
Routing:
- net GND: track 47.3 -> 61.3 mm
- net E_STOP: track 32.8 -> 23.4 mm
- net Net-(J9-Pin_2): track 35.4 -> 26.2 mm
Other:
- board size 148.3 x 76.2 mm -> 94 x 62.1 mm
