File: Wheel V3/_autosave-Wheel V3.kicad_pcb (KiCad board)
At the start: 2 copper layers, 148.3 x 76.2 mm, 63 parts, among them IC1 MT6835GT-STD, J1 Motor_Off, J10 Conn_01x05, J11 Shift Register, J12 MT6835, J13 MT6835, J2 USB_C_Receptacle_USB2.0_16P, J3 Conn_01x07, J4 PWM_OUT, J5 CAN_Connector, J6 I2C_Connector, J7 E-Stop, J8 UART_Connector, J9 TEMP, SW1 SW_Push, SW2 SW_Push, U1 USBLC6-2SC6, U2 LDL111733R-3.3, U3 STM32F407VGTx, Y1 8MHz

Commit message: Update
Parts:
- removed MB5 (x5): 5.5mm, PCM_marbastlib-various:mousebites_5p5mm_easysnap
