File: Wheel V3/brake.kicad_sch (KiCad schematic)
At the start: 15 parts, among them J2 Resistor, J3 PWR, Q1 STP110N8F6, U1 L7812, U2 TC4427xOA, U4 LM393, U5 TL431D

Commit message: Update
Parts:
- C18: renamed from C3; footprint (none) -> Capacitor_SMD:C_0805_2012Metric
- C19: renamed from C4; footprint (none) -> Capacitor_SMD:C_0805_2012Metric
- C20: renamed from C1; footprint (none) -> Capacitor_SMD:C_0805_2012Metric
- C21: renamed from C2; footprint (none) -> Capacitor_SMD:C_0805_2012Metric
- J14: renamed from J3; footprint (none) -> Connector_AMASS:AMASS_XT60-M_1x02_P7.20mm_Vertical
- J15: renamed from J2; footprint (none) -> Connector_AMASS:AMASS_XT60-M_1x02_P7.20mm_Vertical
- Q1: footprint (none) -> Package_TO_SOT_THT:TO-220-3_Vertical
- R16, R17: footprint (none) -> Resistor_SMD:R_0805_2012Metric
- R18: renamed from R19; footprint (none) -> Resistor_SMD:R_0805_2012Metric
- R19: renamed from R18; footprint (none) -> Resistor_SMD:R_0805_2012Metric
- U4: renamed from U1; footprint (none) -> Converter_DCDC:Converter_DCDC_RECOM_R-78E-0.5_THT
- U5: renamed from U4; footprint (none) -> Package_SO:SOIC-8_3.9x4.9mm_P1.27mm
- renumbered U5 to U6, U2 to U7
