File: Wheel Brake/Wheel Brake.kicad_pcb (KiCad board)
At the start: 2 copper layers, 69.9 x 34.8 mm, 18 parts, among them J1 PWR, J2 Resistor, Q1 STP110N8F6, U1 L7812, U2 LM393, U3 TL431D, U4 TC4427xOA

Commit message: Final Update
Connections:
- R1 pad 2: +12V -> Net-(U4-IN_A)
Routing:
- net Net-(U4-IN_A): track 33.2 -> 40.4 mm
- net +12V: track 67.5 -> 60.5 mm
Other:
- board size 69.9 x 34.8 mm -> 59.9 x 27.4 mm
