File: Wheel Brake/Wheel Brake.kicad_sch (KiCad schematic)
At the start: 18 parts, among them J1 PWR, J2 Resistor, Q1 STP110N8F6, U1 L7812, U2 LM393, U3 TL431D, U4 TC4427xOA

Commit message: Final Update
Connections:
- net +12V: no longer R1.2
- net at R4.2, U2.1, U4.2 (IN_A)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: now also R1.2
Changed lines of the file:
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@@
 		(color 0 0 0 0)
 	)
-	(junction
-		(at 130.81 67.31)
-		(diameter 0)
-		(color 0 0 0 0)
-	)
-	(wire
-		(pts
-			(xy 120.65 50.8) (xy 130.81 50.8)
-		)
-		(stroke
-			(width 0)
-			(type default)
-		)
-	)
-	(wire
-		(pts
-			(xy 130.81 50.8) (xy 130.81 67.31)
-		)
-		(stroke
-			(width 0)
-			(type default)
-		)
-	)
 	(wire
 		(pts
@@
 	(wire
 		(pts
+			(xy 120.65 50.8) (xy 123.19 50.8)
+		)
+		(stroke
+			(width 0)
+			(type default)
+		)
+	)
+	(wire
+		(pts
 			(xy 177.8 53.34) (xy 185.42 53.34)
 		)
 		(stroke
+			(width 0)
+			(type default)
+		)
+	)
+	(wire
+		(pts
+			(xy 123.19 50.8) (xy 123.19 67.31)
+		)
+		(stroke
